File: TouchDRO.kicad_pcb (KiCad board)
At the start: 2 copper layers, 55.9 x 55.4 mm, 25 parts, among them J1 X, J2 Y, J3 Z, J4 W, J5 VIN, U2 AM26LV32xD, U3 AM26LV32xD

Commit message: v0.2
Routing:
- net +5V: track 165.6 -> 162.9 mm
- net GND: vias 71 -> 69
Changed lines of the file:
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@@
 		(title "dns' TouchDRO")
 		(date "2025-02-22")
-		(rev "0.1")
+		(rev "0.2")
 	)
 	(layers
@@
 	)
 	(setup
+		(stackup
+			(layer "F.SilkS"
+				(type "Top Silk Screen")
+			)
+			(layer "F.Paste"
+				(type "Top Solder Paste")
+			)
+			(layer "F.Mask"
+				(type "Top Solder Mask")
+				(color "Purple")
+				(thickness 0.01)
+			)
+			(layer "F.Cu"
+				(type "copper")
+				(thickness 0.035)
+			)
+			(layer "dielectric 1"
+				(type "core")
+				(thickness 1.51)
+				(material "FR4")
+				(epsilon_r 4.5)
+				(loss_tangent 0.02)
+			)
+			(layer "B.Cu"
+				(type "copper")
+				(thickness 0.035)
+			)
+			(layer "B.Mask"
+				(type "Bottom Solder Mask")
+				(color "Purple")
+				(thickness 0.01)
+			)
+			(layer "B.Paste"
+				(type "Bottom Solder Paste")
+			)
+			(layer "B.SilkS"
+				(type "Bottom Silk Screen")
+			)
+			(copper_finish "None")
+			(dielectric_constraints no)
+		)
 		(pad_to_mask_clearance 0)
 		(allow_soldermask_bridges_in_footprints no)
@@
 			(drillshape 0)
 			(scaleselection 1)
-			(outputdirectory "gbr/TouchDRO-v0.1/")
+			(outputdirectory "gbr/TouchDRO-v0.2")
 		)
 	)
@@
 	)
 	(via
-		(at 47.117 85.725)
+		(at 47.752 85.725)
 		(size 0.8)
 		(drill 0.4)
@@
 	)
 	(via
-		(at 46.99 53.34)
-		(size 0.8)
-		(drill 0.4)
-		(layers "F.Cu" "B.Cu")
-		(free yes)
-		(net 1)
-	)
-	(via
 		(at 58.674 38.989)
 		(size 0.8)
@@
 	)
 	(via
-		(at 47.117 56.769)
+		(at 47.498 56.642)
 		(size 0.8)
 		(drill 0.4)
@@
 	)
 	(via
-		(at 46.99 82.55)
-		(size 0.8)
-		(drill 0.4)
-		(layers "F.Cu" "B.Cu")
-		(free yes)
-		(net 1)
-	)
-	(via
 		(at 88.646 40.894)
 		(size 0.8)
@@
 	)
 	(via
-		(at 47.879 57.531)
+		(at 47.498 57.912)
 		(size 0.8)
 		(drill 0.4)
@@
 	)
 	(via
-		(at 100.203 73.787)
+		(at 99.822 73.787)
 		(size 0.8)
 		(drill 0.4)
@@
 	)
 	(segment
-		(start 53.2318 86.958)
-		(end 46.697 86.958)
+		(start 46.772 48.478)
+		(end 46.772 74.727)
 		(width 0.25)
 		(layer "B.Cu")
@@
 	)
 	(segment
-		(start 45.972 49.278)
-		(end 45.972 73.927)
+		(start 52.7248 86.451)
+		(end 47.45128 86.451)
 		(width 0.25)
 		(layer "B.Cu")
@@
 	)
 	(segment
-		(start 98.943701 45.212)
-		(end 100.235 46.503299)
+		(start 46.772 74.727)
+		(end 48.255 76.21)
 		(width 0.25)
 		(layer "B.Cu")
@@
 	)
 	(segment
-		(start 45.972 73.927)
-		(end 48.255 76.21)
+		(start 98.943701 45.212)
+		(end 100.235 46.503299)
 		(width 0.25)
 		(layer "B.Cu")
@@
 	)
 	(segment
-		(start 101.348 56.898)
-		(end 99.06 54.61)
+		(start 100.548 56.098)
+		(end 100.548 82.332)
 		(width 0.25)
 		(layer "B.Cu")
@@
 	)
 	(segment
-		(start 99.06 83.82)
-		(end 101.348 81.532)
+		(start 46.736 85.73572)
+		(end 46.736 77.729)
 		(width 0.25)
 		(layer "B.Cu")
@@
 	)
 	(segment
-		(start 45.972 86.233)
-		(end 45.972 78.493)
+		(start 57.409 91.1352)
+		(end 52.7248 86.451)
 		(width 0.25)
 		(layer "B.Cu")
@@
 	)
 	(segment
-		(start 101.348 81.532)
-		(end 101.348 56.898)
+		(start 100.548 82.332)
+		(end 99.06 83.82)
 		(width 0.25)
 		(layer "B.Cu")
@@
 	)
 	(segment
-		(start 48.26 46.99)
-		(end 45.972 49.278)
+		(start 93.520695 41.714)
+		(end 97.018695 45.212)
 		(width 0.25)
 		(layer "B.Cu")
@@
 	)
 	(segment
-		(start 57.409 91.1352)
-		(end 53.2318 86.958)
+		(start 99.06 54.61)
+		(end 100.548 56.098)
 		(width 0.25)
 		(layer "B.Cu")
@@
 	)
 	(segment
-		(start 93.520695 41.714)
-		(end 97.018695 45.212)
+		(start 48.26 46.99)
+		(end 46.772 48.478)
 		(width 0.25)
 		(layer "B.Cu")
@@
 	)
 	(segment
-		(start 46.697 86.958)
-		(end 45.972 86.233)
+		(start 100.235 53.435)
+		(end 99.06 54.61)
 		(width 0.25)
 		(layer "B.Cu")
@@
 	)
 	(segment
-		(start 100.235 53.435)
-		(end 99.06 54.61)
+		(start 97.018695 45.212)
+		(end 98.943701 45.212)
 		(width 0.25)
 		(layer "B.Cu")
@@
 	)
 	(segment
-		(start 97.018695 45.212)
-		(end 98.943701 45.212)
+		(start 47.45128 86.451)
+		(end 46.736 85.73572)
 		(width 0.25)
 		(layer "B.Cu")
@@
 	)
 	(segment
-		(start 45.972 78.493)
+		(start 46.736 77.729)
 		(end 48.255 76.21)
 		(width 0.25)
@@
 		(polygon
 			(pts
-				(xy 45.72 38.1) (xy 101.6 38.1) (xy 101.6 92.71) (xy 45.72 92.71)
+				(xy 45.72 37.846) (xy 101.6 37.846) (xy 101.6 93.218) (xy 45.72 93.218)
 			)
 		)
